File: workspaces/nmos-ldo/kicad/sheets/error-amplifier.kicad_sch (KiCad schematic)
At the start: 0 parts

Commit message: Standardize electrical design contracts and KiCad SPICE workflows
Parts:
- added Q1, Q2, Q3, Q4, Q5, Q6: SKY130_PMOS_LVT_4T, symbol AnalogBench:SKY130_PMOS_LVT_4T
- added Q10, Q11, Q12, Q7, Q8, Q9: SKY130_NMOS_LVT_4T, symbol AnalogBench:SKY130_NMOS_LVT_4T
Connections:
- net ibias: now also Q1.2 (G), Q4.1 (D), Q4.2 (G)
- net loop_out: now also Q10.1 (D), Q6.1 (D)
- net vdd: now also Q1.3 (S), Q1.4 (B), Q2.4 (B), Q3.4 (B), Q4.3 (S), Q4.4 (B), Q5.3 (S), Q5.4 (B), Q6.3 (S), Q6.4 (B)
- net vfb: now also Q2.2 (G)
- net vref: now also Q3.2 (G)
- net vss: now also Q10.3 (S), Q10.4 (B), Q11.3 (S), Q11.4 (B), Q12.3 (S), Q12.4 (B), Q7.3 (S), Q7.4 (B), Q8.3 (S), Q8.4 (B), Q9.3 (S), Q9.4 (B)
- new net nleft: Q11.2 (G), Q12.1 (D), Q2.1 (D), Q7.1 (D), Q7.2 (G), Q9.2 (G)
- new net nright: Q10.2 (G), Q11.1 (D), Q12.2 (G), Q3.1 (D), Q8.1 (D), Q8.2 (G)
- new net pdiag: Q5.1 (D), Q5.2 (G), Q6.2 (G), Q9.1 (D)
- new net ptail: Q1.1 (D), Q2.3 (S), Q3.3 (S)
